File: Source/LORA DEVBOARD.kicad_pcb (KiCad board)
At the start: 4 copper layers, 51.9 x 75 mm, 32 parts, among them J2 Conn_01x13, J3 JST, J4 Conn_01x13, SW1 RKCGG140GSMTRLFS, SW2 RKCGG140GSMTRLFS, U1 ESP32-S3-WROOM-1, U2 SX1262IMLTRT, U3 AMS1117-3.3, U4 TP4056, U5 BWU.FL-IPEX1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

Commit message: Update PCB
Parts:
- added C11: 10uF, Capacitor_SMD:C_0603_1608Metric, F.Cu at (207.5, 67.5)
- added C12: 100nF, Capacitor_SMD:C_0603_1608Metric, F.Cu at (206.0, 67.5)
- moved C4 17.2 mm to (194.3, 110.8)
- moved C8 17.2 mm to (194.3, 112.4)
- moved C9 17.2 mm to (201.9, 111.9)
- moved C10 17.2 mm to (199.4, 114.4)
- moved C5 17.2 mm to (199.1, 103.8)
- moved C7 17.2 mm to (191.3, 110.8)
- moved L1 17.2 mm to (199.1, 106.8)
- moved U5 17.2 mm to (191.6, 107.8)
- moved Y1 17.2 mm to (199.1, 111.6)
- moved C6 17.2 mm to (200.7, 108.1)
- moved U2 17.1 mm to (195.7, 107.0)
- moved C1 14.2 mm to (215.9, 104.2)
- moved C2 14.2 mm to (212.5, 104.2)
- moved C3 14.2 mm to (212.1, 93.3)
- moved U3 14.2 mm to (212.1, 98.7)
Routing:
- net +3.3V: track 159.8 -> 186.7 mm, vias 0 -> 2
- net +5V: track 52.9 -> 76.5 mm
- net DIO1: track 10.2 -> 28.2 mm
- net unconnected-(USB1-PadEP): track 18.3 -> 0.57 mm
- net NRESET: track 46.6 -> 64.1 mm
- net BUSY: track 32.5 -> 48.9 mm
- net NSS: track 18.1 -> 32.9 mm
- net SCK: track 28.1 -> 42.4 mm
- net MISO: track 27.2 -> 39.5 mm
- net MOSI: track 27.6 -> 39.9 mm
- net GND: track 50.8 -> 53.0 mm, vias 35 -> 37
- net GPIO13: track 34.0 -> 36.2 mm
- net GPIO11: track 36.1 -> 35.2 mm
