File: Source/LORA DEVBOARD.kicad_sch (KiCad schematic)
At the start: 28 parts, among them J2 Conn_01x13, J3 JST, J4 Conn_01x13, SW1 RKCGG140GSMTRLFS, SW2 RKCGG140GSMTRLFS, U1 ESP32-S3-WROOM-1, U2 SX1262IMLTRT, U3 AMS1117-3.3, U4 TP4056, U5 BWU.FL-IPEX1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

Commit message: Update PCB
Parts:
- added C11: 10uF, Capacitor_SMD:C_0603_1608Metric, symbol Device:C
- added C12: 100nF, Capacitor_SMD:C_0603_1608Metric, symbol Device:C
Connections:
- net +3.3V: now also C11.2, C12.2
- net GND: now also C11.1, C12.1
