File: Source/KiCAD/LORA DEVBOARD.kicad_pcb (KiCad board)
At the start: 4 copper layers, 51.9 x 75 mm, 34 parts, among them J2 Conn_01x13, J3 JST, J4 Conn_01x13, SW1 RKCGG140GSMTRLFS, SW2 RKCGG140GSMTRLFS, U1 ESP32-S3-WROOM-1, U2 SX1262IMLTRT, U3 AMS1117-3.3, U4 TP4056, U5 BWU.FL-IPEX1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

Commit message: Replace Files
Parts:
- moved REF** 15.9 mm to (192.0, 53.5)
- moved REF** 15.2 mm to (236.0, 53.5)
- moved C12 5.21 mm to (200.8, 67.7)
- moved C11 5.21 mm to (202.3, 67.7)
- moved REF** 5.16 mm to (192.0, 121.2)
- moved REF** 4.64 mm to (236.0, 121.2)
- moved R6 4.40 mm to (217.9, 114.3)
- moved R7 4.40 mm to (211.5, 114.3)
- moved USB1 4.37 mm to (214.1, 119.4)
- moved U1 3.92 mm to (214.1, 75.4)
- moved C1 3.17 mm to (219.0, 104.3)
- moved C2 3.17 mm to (215.6, 104.3)
- moved C3 3.17 mm to (215.3, 93.5)
- moved U3 3.17 mm to (215.2, 98.8)
- moved J4 0.81 mm to (235.1, 99.6)
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Routing:
- net GPIO12: track 76.8 -> 90.2 mm
- net D+: track 81.9 -> 91.8 mm
- net GPIO10: track 44.3 -> 54.0 mm
- net D-: track 79.4 -> 88.0 mm
- net GPIO1: track 16.3 -> 24.1 mm
- net +5V: track 76.5 -> 84.0 mm
- net NRESET: track 64.1 -> 69.1 mm
- net GPIO47: track 37.4 -> 32.7 mm
- net NSS: track 32.9 -> 37.4 mm
- net MISO: track 39.5 -> 35.4 mm
- net BUSY: track 48.9 -> 45.0 mm
- net IO0: track 5.23 -> 9.15 mm
- net GPIO14: track 33.6 -> 29.8 mm
- net SCK: track 42.4 -> 38.6 mm
- net GPIO2: track 11.3 -> 14.9 mm
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